Commit message: add gazebo
Signed-off-by: ijnek <kenjibrameld@gmail.com>

File: urdf/cameras.urdf (robot description, URDF)
Before this commit: robot cameras, 3 links, 2 joints
Links:
- link depth_camera: mass None -> 1.00; geometry collision box size=0.1 0.1 0.1; visual box size=0.1 0.1 0.1
- link rgb_camera: mass None -> 1.00; geometry collision box size=0.1 0.1 0.1; visual box size=0.1 0.1 0.1

Commit message: get rgb image showing in rviz
Signed-off-by: ijnek <kenjibrameld@gmail.com>

File: urdf/cameras.urdf (robot description, URDF)
Before this commit: robot cameras, 3 links, 2 joints
Links:
- added link depth_camera_optical
- added link rgb_camera_optical
Joints:
- added joint depth_camera__depth_camera_optical: type fixed, parent depth_camera, child depth_camera_optical, origin xyz=0 0 0 rpy=-1.57 0 -1.57
- added joint rgb_camera__rgb_camera_optical: type fixed, parent rgb_camera, child rgb_camera_optical, origin xyz=0 0 0 rpy=-1.57 0 -1.57
